File: Quadricoptere/Puissance_quadri/power_dispatch_v1.brd (EAGLE design)
At the start: 50 x 50 mm, 12 parts

Commit message: modification carte quadricoptere
Parts:
- removed C5, C8: 20n, rcl:C1206K
- added C1, C2: 4,7u, SparkFun-Passives:CPOL-RADIAL-10UF-25V
- added C3: 100n, SparkFun-Passives:CAP-PTH-SMALL2
- moved LED1 28.7 mm to (42.1, 3.48), turned to 90 degrees
- moved R1 22.0 mm to (41.1, 11.2), turned to 180 degrees
- moved U$4 16.5 mm to (26.2, 15.0), turned to 90 degrees
- moved R4 5.87 mm to (30.1, 20.6), turned to 90 degrees
- flipped X1 to the top, turned to 90 degrees
- flipped X2 to the top
- flipped X3 to the top, turned to 270 degrees
- flipped X4 to the top, turned to 270 degrees
- flipped X5 to the top
Connections:
- net +5V: now also C2.1, C3.1; no longer C5.1
- net GND: now also C1.2, C2.2, C3.2; no longer C5.2, C8.2
- net VIN: now also C1.1; no longer C8.1
Routing:
- net N$9: track 0.00 -> 17.6 mm
- net N$8: track 0.00 -> 15.4 mm
- net N$4: track 0.00 -> 13.9 mm
- net N$2: track 0.00 -> 13.7 mm
- net N$3: track 0.00 -> 13.5 mm
- net N$11: track 0.00 -> 12.4 mm
- net N$10: track 0.00 -> 12.0 mm
- net N$1: track 0.00 -> 11.5 mm
- net N$6: track 0.00 -> 11.4 mm
- net N$7: track 0.00 -> 10.3 mm
- net N$13: track 0.00 -> 9.88 mm
- net N$12: track 3.02 -> 10.4 mm
- net +5V: track 30.8 -> 26.5 mm
- net GND: track 21.5 -> 17.7 mm
- net N$5: track 4.45 -> 7.46 mm
Other:
- board text removed: "Théo & Cédric"
