File: Quadricoptere/Puissance_quadri/power_dispatch_v1.sch (EAGLE design)
At the start: 12 parts

Commit message: modification carte quadricoptere
Parts:
- removed C5, C8: 20n, rcl:C-EUC1206K
- added C1, C2: 4,7u, SparkFun-Passives:CAP_POLPTH2
- added C3: 100n, SparkFun-Passives:CAPPTH2
Connections:
- net +5V: now also C2.+, C3.1; no longer C5.1
- net GND: now also C1.-, C2.-, C3.2; no longer C5.2, C8.2
- net VIN: now also C1.+; no longer C8.1
Changed lines of the file:
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@@
 <part name="P+9" library="supply1" deviceset="+5V" device=""/>
 <part name="R4" library="rcl" deviceset="R-EU_" device="R0805" value="350"/>
-<part name="C5" library="rcl" deviceset="C-EU" device="C1206K" value="20n"/>
-<part name="C8" library="rcl" deviceset="C-EU" device="C1206K" value="20n"/>
 <part name="X1" library="con-weidmueller-sl35" deviceset="90-2" device=""/>
 <part name="X2" library="con-weidmueller-sl35" deviceset="90-2" device=""/>
@@
 <part name="R1" library="mbed-rlcq" deviceset="R" device="0805" value="1k"/>
 <part name="X6" library="con-molex" deviceset="KK-156-2" device=""/>
+<part name="C1" library="SparkFun-Passives" deviceset="CAP_POL" device="PTH2" value="4,7u"/>
+<part name="C2" library="SparkFun-Passives" deviceset="CAP_POL" device="PTH2" value="4,7u"/>
+<part name="C3" library="SparkFun-Passives" deviceset="CAP" device="PTH2" value="100n"/>
 </parts>
 <sheets>
@@
 <instance part="P+9" gate="1" x="73.66" y="73.66"/>
 <instance part="R4" gate="G$1" x="71.12" y="40.64" rot="R90"/>
-<instance part="C5" gate="G$1" x="78.74" y="50.8"/>
-<instance part="C8" gate="G$1" x="43.18" y="40.64"/>
 <instance part="X1" gate="G$1" x="127" y="68.58"/>
 <instance part="X2" gate="G$1" x="127" y="60.96"/>
@@
 <instance part="X6" gate="-1" x="124.46" y="35.56"/>
 <instance part="X6" gate="-2" x="124.46" y="30.48"/>
+<instance part="C1" gate="G$1" x="43.18" y="40.64"/>
+<instance part="C2" gate="G$1" x="78.74" y="50.8"/>
+<instance part="C3" gate="G$1" x="86.36" y="43.18"/>
 </instances>
 <busses>
@@
 <wire x1="68.58" y1="53.34" x2="73.66" y2="53.34" width="0.1524" layer="91"/>
 <wire x1="73.66" y1="53.34" x2="73.66" y2="63.5" width="0.1524" layer="91"/>
-<pinref part="C5" gate="G$1" pin="1"/>
 <wire x1="73.66" y1="63.5" x2="73.66" y2="71.12" width="0.1524" layer="91"/>
 <wire x1="73.66" y1="53.34" x2="78.74" y2="53.34" width="0.1524" layer="91"/>
@@
 <pinref part="R1" gate="G$1" pin="P$2"/>
 <wire x1="96.52" y1="63.5" x2="73.66" y2="63.5" width="0.1524" layer="91"/>
+<pinref part="C2" gate="G$1" pin="+"/>
+<pinref part="C3" gate="G$1" pin="1"/>
+<wire x1="86.36" y1="48.26" x2="86.36" y2="53.34" width="0.1524" layer="91"/>
+<wire x1="86.36" y1="53.34" x2="78.74" y2="53.34" width="0.1524" layer="91"/>
 </segment>
 <segment>
@@
 <pinref part="R4" gate="G$1" pin="1"/>
 <wire x1="71.12" y1="35.56" x2="58.42" y2="35.56" width="0.1524" layer="91"/>
-<pinref part="C8" gate="G$1" pin="2"/>
-<pinref part="C5" gate="G$1" pin="2"/>
 <wire x1="43.18" y1="35.56" x2="58.42" y2="35.56" width="0.1524" layer="91"/>
 <wire x1="78.74" y1="45.72" x2="78.74" y2="35.56" width="0.1524" layer="91"/>
@@
 <pinref part="LED1" gate="G$1" pin="C"/>
 <wire x1="96.52" y1="43.18" x2="96.52" y2="35.56" width="0.1524" layer="91"/>
-<wire x1="96.52" y1="35.56" x2="78.74" y2="35.56" width="0.1524" layer="91"/>
+<wire x1="96.52" y1="35.56" x2="86.36" y2="35.56" width="0.1524" layer="91"/>
+<pinref part="C1" gate="G$1" pin="-"/>
+<pinref part="C2" gate="G$1" pin="-"/>
+<pinref part="C3" gate="G$1" pin="2"/>
+<wire x1="86.36" y1="35.56" x2="78.74" y2="35.56" width="0.1524" layer="91"/>
+<wire x1="86.36" y1="40.64" x2="86.36" y2="35.56" width="0.1524" layer="91"/>
 </segment>
 <segment>
@@
 <wire x1="50.8" y1="53.34" x2="48.26" y2="53.34" width="0.1524" layer="91"/>
 <wire x1="48.26" y1="53.34" x2="48.26" y2="55.88" width="0.1524" layer="91"/>
-<pinref part="C8" gate="G$1" pin="1"/>
 <wire x1="48.26" y1="53.34" x2="43.18" y2="53.34" width="0.1524" layer="91"/>
 <wire x1="43.18" y1="53.34" x2="43.18" y2="43.18" width="0.1524" layer="91"/>
@@
 <wire x1="48.26" y1="53.34" x2="48.26" y2="66.04" width="0.1524" layer="91"/>
 <label x="40.64" y="60.96" size="1.778" layer="95"/>
+<pinref part="C1" gate="G$1" pin="+"/>
 </segment>
 <segment>
